Commit message: point clouds

File: urdf/d435_gazebo_sim.urdf.xacro (robot description, xacro)
@@ -26,12 +26,18 @@
     name="camera"
     use_nominal_extrinsics="true"
-    use_mesh="false">
+    use_mesh="true">
     <origin xyz="0 0 0" rpy="0 0 0"/>
   </xacro:sensor_d435>
   <!-- ========== GAZEBO SIM SENSORS (New API) ========== -->
-  <!-- Camera link material for Gazebo -->
-  <!--gazebo reference="camera_link">
-    <material>Gazebo/DarkGrey</material>
-  </gazebo-->
+  <!-- Camera link material for Gazebo Sim (Harmonic) -->
+  <gazebo reference="camera_link">
+    <visual>
+      <material>
+        <ambient>0.1 0.1 0.1 1</ambient>
+        <diffuse>0.3 0.3 0.35 1</diffuse>
+        <specular>0.2 0.2 0.2 1</specular>
+      </material>
+    </visual>
+  </gazebo>
   <!-- RGB Camera Sensor -->
   <gazebo reference="camera_color_frame">
@@ -61,7 +67,7 @@
     </sensor>
   </gazebo>
-  <!-- Depth Camera Sensor -->
-  <gazebo reference="camera_depth_optical_frame">
-    <sensor name="camera_depth" type="depth_camera">
+  <!-- RGBD Camera Sensor (publishes depth image + point cloud) -->
+  <gazebo reference="camera_depth_frame">
+    <sensor name="camera_rgbd" type="rgbd_camera">
       <update_rate>30</update_rate>
       <camera>
@@ -70,5 +76,5 @@
           <width>640</width>
           <height>480</height>
-          <format>R_FLOAT32</format>
+          <format>R8G8B8</format>
         </image>
         <clip>
@@ -79,10 +85,10 @@
           <type>gaussian</type>
           <mean>0.0</mean>
-          <stddev>0.1</stddev>
+          <stddev>0.007</stddev>
         </noise>
       </camera>
       <always_on>1</always_on>
       <visualize>false</visualize>
-      <topic>camera/depth/image_raw</topic>
+      <topic>camera/rgbd</topic>
     </sensor>
   </gazebo>
